Commit message: refactor: update Livox SDK2 core components, driver configurations, and third-party dependencies

File: src/ugv_main/ugv_description/urdf/ugv_rover.urdf (robot description, URDF)
Before this commit: robot ugv_rover, 13 links, 12 joints
Links:
- removed link base_lidar_link
Joints:
- removed joint base_lidar_link_joint
- joint 3d_camera_link_joint: origin xyz=0.06531 0 0.021953 rpy=0 0 0 -> xyz=0.06531 0 0.021953 rpy=-1.5708 0 -1.5708

File: src/ugv_main/ugv_gazebo/urdf/ugv_rover.urdf (robot description, URDF)
Before this commit: robot ugv_rover, 13 links, 12 joints
Links:
- removed link base_lidar_link
Joints:
- removed joint base_lidar_link_joint
