Commit message: feat: replace laser scanner with Livox Mid360 lidar in model and URDF

File: src/ugv_main/ugv_gazebo/urdf/rasp_rover.urdf (robot description, URDF)
Before this commit: robot rasp_rover, 12 links, 11 joints
Links:
- removed link base_lidar_link
Joints:
- removed joint base_lidar_link_joint

Commit message: Replace 2D LiDAR with Livox MID-360 on UGV and Rasp Rover

File: src/ugv_main/ugv_gazebo/urdf/rasp_rover.urdf (robot description, URDF)
Before this commit: robot rasp_rover, 11 links, 10 joints
Links:
- added link livox, mass 0.01
Joints:
- added joint livox_joint: type fixed, parent base_link, child livox, origin xyz=-0.05 0 0.08 rpy=0 0 0

File: src/ugv_main/ugv_gazebo/urdf/ugv_rover.urdf (robot description, URDF)
Before this commit: robot ugv_rover, 12 links, 11 joints
Links:
- added link livox, mass 0.01
Joints:
- added joint livox_joint: type fixed, parent base_link, child livox, origin xyz=-0.05 0 0.08 rpy=0 0 0
