Commit message: Align Waver workspace execution with jo branch

File: src/ugv_main/ugv_gazebo/urdf/mid360.xacro (robot description, xacro)
@@ -4,5 +4,5 @@
   <xacro:property name="laser_min_range" value="0.1"/>
   <xacro:property name="laser_max_range" value="200.0"/>
-  <xacro:property name="samples" value="40000"/>
+  <xacro:property name="samples" value="80000"/>
   <xacro:property name="resolution" value="0.002"/>
   <xacro:property name="noise_mean" value="0.0"/>

Commit message: Integrate ros2_ws3 Gazebo SEO patrol workflow

File: src/ugv_main/ugv_gazebo/urdf/mid360.xacro (robot description, xacro)
@@ -4,5 +4,5 @@
   <xacro:property name="laser_min_range" value="0.1"/>
   <xacro:property name="laser_max_range" value="200.0"/>
-  <xacro:property name="samples" value="80000"/>
+  <xacro:property name="samples" value="5000"/>
   <xacro:property name="resolution" value="0.002"/>
   <xacro:property name="noise_mean" value="0.0"/>
